File: 5vFanDriver/5vFanDriver.kicad_pcb (KiCad board)
At the start: 2 copper layers, 18.5 x 26.2 mm, 10 parts, among them J1 Conn_02x03_Odd_Even, J2 Conn_01x04_Male, Q1 2N3904, Q2 2N3904, Q3 2N3906, Q4 2N3906

Commit message: Updating some of these.
Parts:
- moved Q4 0.44 mm to (68.3, 64.0)
Routing:
- net Net-(J1-Pad3): track 27.4 -> 28.1 mm
Other:
- net class Default: via_dia 0.8 -> 1; via_drill 0.4 -> 0.7

Commit message: Updated quite a few things. I've lost count. I think this is the RAMBo cover.
Parts:
- J2: footprint Connector_PinHeader_2.00mm:PinHeader_1x04_P2.00mm_Vertical -> Connector_PinHeader_2.54mm:PinHeader_1x04_P2.54mm_Vertical
- moved J2 0.61 mm to (69.8, 73.7)
Routing:
- net Net-(J2-Pad4): track 12.7 -> 11.8 mm
- net Net-(J2-Pad1): track 12.1 -> 12.6 mm
Changed lines of the file:
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@@
     (thickness 1.5)
     (drawings 11)
-    (tracks 76)
+    (tracks 78)
     (zones 0)
     (modules 10)
@@
     (0 F.Cu signal)
     (31 B.Cu signal)
-    (34 B.Paste user)
+    (34 B.Paste user hide)
     (35 F.Paste user)
-    (36 B.SilkS user)
-    (37 F.SilkS user hide)
-    (38 B.Mask user)
-    (39 F.Mask user hide)
+    (36 B.SilkS user hide)
+    (37 F.SilkS user)
+    (38 B.Mask user hide)
+    (39 F.Mask user)
     (44 Edge.Cuts user)
     (45 Margin user)
@@
     (47 F.CrtYd user)
     (48 B.Fab user)
-    (49 F.Fab user hide)
+    (49 F.Fab user)
   )
   (setup
@@
     (add_net "Net-(Q4-Pad2)")
   )
+  (module Connector_PinHeader_2.54mm:PinHeader_1x04_P2.54mm_Vertical (layer F.Cu)
+    (at 69.85 73.66 90)
+    (descr "Through hole straight pin header, 1x04, 2.54mm pitch, single row")
+    (tags "Through hole pin header THT 1x04 2.54mm single row")
+    (fp_text reference J2 (at 0 -2.33 90) (layer F.SilkS)
+      (effects (font (size 1 1) (thickness 0.15)))
+    )
+    (fp_text value Conn_01x04_Male (at 0 9.95 90) (layer F.Fab)
+      (effects (font (size 1 1) (thickness 0.15)))
+    )
+    (fp_line (start -0.635 -1.27) (end 1.27 -1.27) (layer F.Fab) (width 0.1))
+    (fp_line (start 1.27 -1.27) (end 1.27 8.89) (layer F.Fab) (width 0.1))
+    (fp_line (start 1.27 8.89) (end -1.27 8.89) (layer F.Fab) (width 0.1))
+    (fp_line (start -1.27 8.89) (end -1.27 -0.635) (layer F.Fab) (width 0.1))
+    (fp_line (start -1.27 -0.635) (end -0.635 -1.27) (layer F.Fab) (width 0.1))
+    (fp_line (start -1.33 8.95) (end 1.33 8.95) (layer F.SilkS) (width 0.12))
+    (fp_line (start -1.33 1.27) (end -1.33 8.95) (layer F.SilkS) (width 0.12))
+    (fp_line (start 1.33 1.27) (end 1.33 8.95) (layer F.SilkS) (width 0.12))
+    (fp_line (start -1.33 1.27) (end 1.33 1.27) (layer F.SilkS) (width 0.12))
+    (fp_line (start -1.33 0) (end -1.33 -1.33) (layer F.SilkS) (width 0.12))
+    (fp_line (start -1.33 -1.33) (end 0 -1.33) (layer F.SilkS) (width 0.12))
+    (fp_line (start -1.8 -1.8) (end -1.8 9.4) (layer F.CrtYd) (width 0.05))
+    (fp_line (start -1.8 9.4) (end 1.8 9.4) (layer F.CrtYd) (width 0.05))
+    (fp_line (start 1.8 9.4) (end 1.8 -1.8) (layer F.CrtYd) (width 0.05))
+    (fp_line (start 1.8 -1.8) (end -1.8 -1.8) (layer F.CrtYd) (width 0.05))
+    (fp_text user %R (at 0 3.81 180) (layer F.Fab)
+      (effects (font (size 1 1) (thickness 0.15)))
+    )
+    (pad 1 thru_hole rect (at 0 0 90) (size 1.7 1.7) (drill 1) (layers *.Cu *.Mask)
+      (net 12 "Net-(J2-Pad1)"))
+    (pad 2 thru_hole oval (at 0 2.54 90) (size 1.7 1.7) (drill 1) (layers *.Cu *.Mask)
+      (net 9 "Net-(J1-Pad2)"))
+    (pad 3 thru_hole oval (at 0 5.08 90) (size 1.7 1.7) (drill 1) (layers *.Cu *.Mask)
+      (net 9 "Net-(J1-Pad2)"))
+    (pad 4 thru_hole oval (at 0 7.62 90) (size 1.7 1.7) (drill 1) (layers *.Cu *.Mask)
+      (net 11 "Net-(J2-Pad4)"))
+    (model ${KISYS3DMOD}/Connector_PinHeader_2.54mm.3dshapes/PinHeader_1x04_P2.54mm_Vertical.wrl
+      (at (xyz 0 0 0))
+      (scale (xyz 1 1 1))
+      (rotate (xyz 0 0 0))
+    )
+  )
   (module Package_TO_SOT_THT:TO-92_HandSolder (layer B.Cu)
     (at 68.326 64.008 180)
@@
       (net 12 "Net-(J2-Pad1)"))
     (model ${KISYS3DMOD}/Package_TO_SOT_THT.3dshapes/TO-92.wrl
-      (at (xyz 0 0 0))
-      (scale (xyz 1 1 1))
-      (rotate (xyz 0 0 0))
-    )
-  )
-  (module Connector_PinHeader_2.00mm:PinHeader_1x04_P2.00mm_Vertical (layer F.Cu)
-    (at 70.302 74.07 90)
-    (descr "Through hole straight pin header, 1x04, 2.00mm pitch, single row")
-    (tags "Through hole pin header THT 1x04 2.00mm single row")
-    (fp_text reference J2 (at 0 -2.06 90) (layer F.SilkS)
-      (effects (font (size 1 1) (thickness 0.15)))
-    )
-    (fp_text value Conn_01x04_Male (at 0 8.06 90) (layer F.Fab)
-      (effects (font (size 1 1) (thickness 0.15)))
-    )
-    (fp_line (start -0.5 -1) (end 1 -1) (layer F.Fab) (width 0.1))
-    (fp_line (start 1 -1) (end 1 7) (layer F.Fab) (width 0.1))
-    (fp_line (start 1 7) (end -1 7) (layer F.Fab) (width 0.1))
-    (fp_line (start -1 7) (end -1 -0.5) (layer F.Fab) (width 0.1))
-    (fp_line (start -1 -0.5) (end -0.5 -1) (layer F.Fab) (width 0.1))
-    (fp_line (start -1.06 7.06) (end 1.06 7.06) (layer F.SilkS) (width 0.12))
-    (fp_line (start -1.06 1) (end -1.06 7.06) (layer F.SilkS) (width 0.12))
-    (fp_line (start 1.06 1) (end 1.06 7.06) (layer F.SilkS) (width 0.12))
-    (fp_line (start -1.06 1) (end 1.06 1) (layer F.SilkS) (width 0.12))
-    (fp_line (start -1.06 0) (end -1.06 -1.06) (layer F.SilkS) (width 0.12))
-    (fp_line (start -1.06 -1.06) (end 0 -1.06) (layer F.SilkS) (width 0.12))
-    (fp_line (start -1.5 -1.5) (end -1.5 7.5) (layer F.CrtYd) (width 0.05))
-    (fp_line (start -1.5 7.5) (end 1.5 7.5) (layer F.CrtYd) (width 0.05))
-    (fp_line (start 1.5 7.5) (end 1.5 -1.5) (layer F.CrtYd) (width 0.05))
-    (fp_line (start 1.5 -1.5) (end -1.5 -1.5) (layer F.CrtYd) (width 0.05))
-    (fp_text user %R (at 0 3 180) (layer F.Fab)
-      (effects (font (size 1 1) (thickness 0.15)))
-    )
-    (pad 1 thru_hole rect (at 0 0 90) (size 1.35 1.35) (drill 0.8) (layers *.Cu *.Mask)
-      (net 12 "Net-(J2-Pad1)"))
-    (pad 2 thru_hole oval (at 0 2 90) (size 1.35 1.35) (drill 0.8) (layers *.Cu *.Mask)
-      (net 9 "Net-(J1-Pad2)"))
-    (pad 3 thru_hole oval (at 0 4 90) (size 1.35 1.35) (drill 0.8) (layers *.Cu *.Mask)
-      (net 9 "Net-(J1-Pad2)"))
-    (pad 4 thru_hole oval (at 0 6 90) (size 1.35 1.35) (drill 0.8) (layers *.Cu *.Mask)
-      (net 11 "Net-(J2-Pad4)"))
-    (model ${KISYS3DMOD}/Connector_PinHeader_2.00mm.3dshapes/PinHeader_1x04_P2.00mm_Vertical.wrl
       (at (xyz 0 0 0))
       (scale (xyz 1 1 1))
@@
   (segment (start 70.866 58.79959) (end 70.866 60.198) (width 0.35) (layer F.Cu) (net 10))
   (segment (start 72.262 54.53) (end 70.946 54.53) (width 0.35) (layer F.Cu) (net 10))
-  (segment (start 78.994 71.378) (end 76.302 74.07) (width 0.35) (layer B.Cu) (net 11) (status 20))
+  (segment (start 78.994 71.374) (end 78.994 72.136) (width 0.35) (layer B.Cu) (net 11))
+  (segment (start 78.802 63.07) (end 78.74 63.132) (width 0.35) (layer B.Cu) (net 11))
+  (segment (start 78.74 63.132) (end 78.74 66.04) (width 0.35) (layer B.Cu) (net 11))
+  (segment (start 78.74 66.04) (end 79.502 66.802) (width 0.35) (layer B.Cu) (net 11))
   (segment (start 79.502 70.866) (end 78.994 71.374) (width 0.35) (layer B.Cu) (net 11))
-  (segment (start 78.802 63.07) (end 78.74 63.132) (width 0.35) (layer B.Cu) (net 11) (status 30))
-  (segment (start 78.994 71.374) (end 78.994 71.378) (width 0.35) (layer B.Cu) (net 11))
-  (segment (start 78.74 63.132) (end 78.74 66.04) (width 0.35) (layer B.Cu) (net 11) (status 10))
   (segment (start 79.502 66.802) (end 79.502 70.866) (width 0.35) (layer B.Cu) (net 11))
-  (segment (start 78.74 66.04) (end 79.502 66.802) (width 0.35) (layer B.Cu) (net 11))
+  (segment (start 78.994 72.136) (end 77.47 73.66) (width 0.35) (layer B.Cu) (net 11))
   (segment (start 69.277 74.07) (end 70.302 74.07) (width 0.35) (layer B.Cu) (net 12))
   (segment (start 68.326 64.008) (end 68.326 65.278) (width 0.35) (layer B.Cu) (net 12))
   (segment (start 68.326 65.278) (end 67.564 66.04) (width 0.35) (layer B.Cu) (net 12))
-  (segment (start 67.564 72.357) (end 69.277 74.07) (width 0.35) (layer B.Cu) (net 12))
   (segment (start 67.564 66.04) (end 67.564 72.357) (width 0.35) (layer B.Cu) (net 12))
+  (segment (start 68.65 73.66) (end 67.564 72.574) (width 0.35) (layer B.Cu) (net 12))
+  (segment (start 67.564 72.574) (end 67.564 72.357) (width 0.35) (layer B.Cu) (net 12))
+  (segment (start 69.85 73.66) (end 68.65 73.66) (width 0.35) (layer B.Cu) (net 12))
 )
