File: 5vFanDriver/5vFanDriver.sch (KiCad schematic (older format))
At the start: 10 parts, among them J1 Conn_02x03_Odd_Even, J2 Conn_01x04_Male, Q1 2N3904, Q2 2N3904, Q3 2N3906, Q4 2N3906

Commit message: Updated quite a few things. I've lost count. I think this is the RAMBo cover.
Parts:
- J2: footprint Connector_PinHeader_2.00mm:PinHeader_1x04_P2.00mm_Vertical -> Connector_PinHeader_2.54mm:PinHeader_1x04_P2.54mm_Vertical
Changed lines of the file:
@@
 F 0 "J2" H 4323 1580 50  0000 R CNN
 F 1 "Conn_01x04_Male" H 4323 1671 50  0000 R CNN
-F 2 "Connector_PinHeader_2.00mm:PinHeader_1x04_P2.00mm_Vertical" H 4350 1700 50  0001 C CNN
+F 2 "Connector_PinHeader_2.54mm:PinHeader_1x04_P2.54mm_Vertical" H 4350 1700 50  0001 C CNN
 F 3 "~" H 4350 1700 50  0001 C CNN
 	1    4350 1700
